Commit message: 제어: 조향 응답 반영 + 경로 헤딩 정렬 기동(ALIGN)
STM32 업링크가 미구현(uart_protocol.md v2 §State)이라 실측 조향각이 없다.
조향각 오차는 곧 곡률 오차이고 곧 경로 이탈이므로, 피드백 없이도 모델이 맞도록
'액추에이터가 따라올 수 있는 속도로만 명령' 하는 쪽으로 정리했다.

조향 응답
  · 조향 슬루 제한 + cmd_vel 재정합 — 제한된 조향각에서 나올 wz 를 역산해
    McuCommand 의 두 필드가 서로 다른 이야기를 하지 않게 했다 (정합오차 2.6e-9 rad/s)
  · 기동 조향 정렬 dwell / 모드 전환 dwell — 조향각을 모르는 구간은 속도 0
  · mode_switch_dwell_sec 3.0 -> 4.0. 기구학이 정한 값이다:
    최악 스윕 normal 풀락(30°) -> spin 제로턴(47°) = 77°, ÷20 deg/s = 3.85 s
  · 정지 2등급 분리 — e-stop/fault=즉시, cmd timeout/odom stale=감속 램프
  · 업링크 부재를 기동 시 1회 알림 (expect_mcu_state=false 가 기본)

ALIGN (신규 path_align.py)
  전역 플래너는 R_min 원호/직선만 이어 붙여 제자리 회전을 표현하지 못한다.
  기존 spin 진입 조건(|wz|>=0.35 and lin<=0.04)은 Nav2 twist 의 사후 분류라,
  플래너가 그런 명령을 낼 이유가 없어 사실상 BT 리커버리 때만 발동했다.

  ALIGN 은 /plan 을 직접 구독해 경로가 요구하는 헤딩과 60° 넘게(0.6 s 지속)
  벌어지면 목표 헤딩을 절대각으로 래치하고 spin 으로 정정 후 normal 로 복귀한다.
  모드 분류가 아니라 '기동'인 것이 핵심이다 — 예전 반경기반 라우팅은 spin 이
  되면 vx=0 이 되어 조건이 자기부정을 일으켜 1틱 단위로 왕복했다.

  · 문턱 60° 는 실측 분포 근거 (경로 추종 중 헤딩오차 p90 9.7°,
    30° 로 낮추면 정상 주행 틱의 35% 가 걸린다)
  · 헤딩오차를 '경로 pose 의 yaw' 로 정의 — 방위각 정의는 후진 구간에서
    p90 173.9° 로 뒤집힌다
  · 자체 시험 19항목: python3 path_align.py
  · 로봇 자세는 TF(map->base_link). /Odometry 는 odom 프레임이라 /plan 과
    직접 비교하면 map->odom 오프셋만큼 통째로 틀어진다

기타
  · fake_mcu 조향 액추에이터 모델(슬루+지연) + 실제 조향각으로 데드레커닝
  · URDF 휠베이스/윤거를 STM32 CONS 기준으로 정정
  · steering_observer 신규 — κ=Δθ/Δs 로 실효 조향각 역산 (업링크 불필요)

상세: docs/control_pipeline.md §6.1~6.3, §6.8

Co-Authored-By: Claude Opus 5 <noreply@anthropic.com>

File: ALM_auto_ws/src/alm_description/urdf/alm_robot.urdf.xacro (robot description, xacro)
@@ -20,8 +20,23 @@
   <xacro:property name="wheel_width"  value="0.0488"/>    <!-- 48.8 mm -->
   <!-- 바퀴 중심 위치 (base_link=차체중심 기준). 앞/뒤 x가 대칭이 아님(CAD 값). -->
-  <xacro:property name="front_x" value="0.6106"/>   <!-- 앞축: FL/RL 평균 X -->
-  <xacro:property name="rear_x"  value="-0.3010"/>  <!-- 뒤축: FR/RR 평균 X -->
-  <xacro:property name="half_track" value="0.500"/> <!-- 좌우 ±500 mm → 트레드 1000 mm -->
-  <!-- 휠베이스 = front_x - rear_x = 0.9116 m (≈912 mm) -->
+  <!--
+    ★ 2026-08-20: STM32 CONS 가 정답임이 확인되어 그 값에 맞춤.
+      이전:  front_x 0.6106 · rear_x -0.3010 · half_track 0.500
+             -> 휠베이스 0.9116 m, 윤거 1.000 m
+      CONS:  CONS(2) 휠베이스 1.000 m,  CONS(3) 윤거 0.919 m
+      두 값이 **뒤바뀌어 적힌** 것으로 보인다:
+        이전 URDF 윤거     1.0000 m  ==  CONS 휠베이스 1.000 m  (정확히 일치)
+        이전 URDF 휠베이스 0.9116 m  ~=  CONS 윤거     0.919 m  (차이 7 mm)
+    ##CONFIRM## front_x / rear_x 배분은 CAD 확인이 필요하다. 휠베이스 합(1.000 m)만
+      CONS 로 확정됐고, base_link 가 축 사이 어디인지는 CONS 에 정보가 없다.
+      아래는 **footprint 를 바꾸지 않는** 안을 택했다 (front_x 유지, rear_x 를 뒤로):
+      앞쪽 최전방 x 가 그대로라 기존 footprint x[-0.65, +0.72] 가 계속 유효하고
+      안전 여유가 줄지 않는다. 배분이 다르면 이 두 줄과 nav2.yaml footprint 를
+      함께 고칠 것.  검사: ros2 run alm_navigation nav2_kinematic_check.py (§6)
+  -->
+  <xacro:property name="front_x" value="0.6106"/>   <!-- 앞축: FL/FR 평균 X (유지) -->
+  <xacro:property name="rear_x"  value="-0.3894"/>  <!-- 뒤축: RL/RR 평균 X (CONS 휠베이스 1.000) -->
+  <xacro:property name="half_track" value="0.4595"/><!-- 좌우 ±459.5 mm -> 윤거 919 mm = CONS(3) -->
+  <!-- 휠베이스 = front_x - rear_x = 1.0000 m = CONS(2) -->
   <!-- 조향 기계적 한계: toe-in 90°, toe-out 45° (URDF 조인트는 시각화용으로 ±90°) -->
   <xacro:property name="steer_lower" value="-1.5708"/>
